File: Hardware/PumpkinPi.sch (KiCad schematic (older format))
At the start: 2 parts

Commit message: wiring progress
Parts:
- added J?: Micro_SD_Card, symbol Connector:Micro_SD_Card
- U?: symbol PumpkinPi:F1C100s -> PumpkinPi-rescue:F1C100s-PumpkinPi
Connections:
- net labels added: +1V1, +2V5, +3V3, SD0_CLK, SD0_CMD, SD0_D0, SD0_D1, SD0_D2, SD0_D3
- no-connect marks 45 -> 42
Changed lines of the file:
@@
 $EndDescr
 $Comp
-L PumpkinPi:F1C100s U?
+L PumpkinPi-rescue:F1C100s-PumpkinPi U?
 U 1 1 60F0B7C1
 P 3550 2950
-F 0 "U?" H 5294 2996 50  0000 L CNN
-F 1 "F1C100s" H 5294 2905 50  0000 L CNN
+F 0 "U?" H 4600 2950 50  0000 L CNN
+F 1 "F1C100s" H 4550 3150 50  0000 L CNN
 F 2 "" H 3550 2900 50  0001 C CNN
 F 3 "" H 3550 2900 50  0001 C CNN
@@
 NoConn ~ 3200 1250
 NoConn ~ 3000 1250
-NoConn ~ 5250 3100
-NoConn ~ 5250 2900
 NoConn ~ 4100 4650
 NoConn ~ 4200 4650
@@
 NoConn ~ 1850 3800
 NoConn ~ 1850 3900
-NoConn ~ 1850 4000
 NoConn ~ 3100 4650
 NoConn ~ 3000 4650
@@
 NoConn ~ 3500 1250
 NoConn ~ 3400 1250
+Text Label 5250 2700 0    50   ~ 0
+SD0_D1
+Text Label 5250 2800 0    50   ~ 0
+SD0_D0
+Text Label 5250 2900 0    50   ~ 0
+SD0_CLK
+Text Label 5250 3000 0    50   ~ 0
+SD0_CMD
+Text Label 5250 3100 0    50   ~ 0
+SD0_D3
+Text Label 5250 3200 0    50   ~ 0
+SD0_D2
+$Comp
+L Connector:Micro_SD_Card J?
+U 1 1 60F0D183
+P 7000 2900
+F 0 "J?" H 6950 3617 50  0000 C CNN
+F 1 "Micro_SD_Card" H 6950 3526 50  0000 C CNN
+F 2 "" H 8150 3200 50  0001 C CNN
+F 3 "http://katalog.we-online.de/em/datasheet/693072010801.pdf" H 7000 2900 50  0001 C CNN
+	1    7000 2900
+	1    0    0    -1
+$EndComp
+Text Label 6100 3200 2    50   ~ 0
+SD0_D0
+Text Label 6100 3300 2    50   ~ 0
+SD0_D1
+Text Label 6100 3000 2    50   ~ 0
+SD0_CLK
+Text Label 6100 2800 2    50   ~ 0
+SD0_CMD
+Text Label 6100 2700 2    50   ~ 0
+SD0_D3
+Text Label 6100 2600 2    50   ~ 0
+SD0_D2
+$Comp
+L power:GND #PWR?
+U 1 1 60F13818
+P 6100 3100
+F 0 "#PWR?" H 6100 2850 50  0001 C CNN
+F 1 "GND" V 6105 2972 50  0000 R CNN
+F 2 "" H 6100 3100 50  0001 C CNN
+F 3 "" H 6100 3100 50  0001 C CNN
+	1    6100 3100
+	0    1    1    0
+$EndComp
+$Comp
+L power:+1V1 #PWR?
+U 1 1 60F16DA1
+P 1850 4000
+F 0 "#PWR?" H 1850 3850 50  0001 C CNN
+F 1 "+1V1" V 1865 4128 50  0000 L CNN
+F 2 "" H 1850 4000 50  0001 C CNN
+F 3 "" H 1850 4000 50  0001 C CNN
+	1    1850 4000
+	0    -1   -1   0
+$EndComp
+$Comp
+L power:+1V1 #PWR?
+U 1 1 60F18349
+P 3700 4650
+F 0 "#PWR?" H 3700 4500 50  0001 C CNN
+F 1 "+1V1" H 3715 4823 50  0000 C CNN
+F 2 "" H 3700 4650 50  0001 C CNN
+F 3 "" H 3700 4650 50  0001 C CNN
+	1    3700 4650
+	-1   0    0    1
+$EndComp
+$Comp
+L power:+2V5 #PWR?
+U 1 1 60F1886B
+P 3200 4650
+F 0 "#PWR?" H 3200 4500 50  0001 C CNN
+F 1 "+2V5" H 3215 4823 50  0000 C CNN
+F 2 "" H 3200 4650 50  0001 C CNN
+F 3 "" H 3200 4650 50  0001 C CNN
+	1    3200 4650
+	-1   0    0    1
+$EndComp
+$Comp
+L power:+2V5 #PWR?
+U 1 1 60F1908B
+P 3300 4650
+F 0 "#PWR?" H 3300 4500 50  0001 C CNN
+F 1 "+2V5" H 3315 4823 50  0000 C CNN
+F 2 "" H 3300 4650 50  0001 C CNN
+F 3 "" H 3300 4650 50  0001 C CNN
+	1    3300 4650
+	-1   0    0    1
+$EndComp
+$Comp
+L power:+2V5 #PWR?
+U 1 1 60F1984F
+P 3400 4650
+F 0 "#PWR?" H 3400 4500 50  0001 C CNN
+F 1 "+2V5" H 3415 4823 50  0000 C CNN
+F 2 "" H 3400 4650 50  0001 C CNN
+F 3 "" H 3400 4650 50  0001 C CNN
+	1    3400 4650
+	-1   0    0    1
+$EndComp
+$Comp
+L power:+2V5 #PWR?
+U 1 1 60F19C7B
+P 3600 4650
+F 0 "#PWR?" H 3600 4500 50  0001 C CNN
+F 1 "+2V5" H 3615 4823 50  0000 C CNN
+F 2 "" H 3600 4650 50  0001 C CNN
+F 3 "" H 3600 4650 50  0001 C CNN
+	1    3600 4650
+	-1   0    0    1
+$EndComp
+$Comp
+L power:+2V5 #PWR?
+U 1 1 60F1A0CF
+P 3800 4650
+F 0 "#PWR?" H 3800 4500 50  0001 C CNN
+F 1 "+2V5" H 3815 4823 50  0000 C CNN
+F 2 "" H 3800 4650 50  0001 C CNN
+F 3 "" H 3800 4650 50  0001 C CNN
+	1    3800 4650
+	-1   0    0    1
+$EndComp
+$Comp
+L power:+1V1 #PWR?
+U 1 1 60F1CAEE
+P 4200 1250
+F 0 "#PWR?" H 4200 1100 50  0001 C CNN
+F 1 "+1V1" H 4215 1423 50  0000 C CNN
+F 2 "" H 4200 1250 50  0001 C CNN
+F 3 "" H 4200 1250 50  0001 C CNN
+	1    4200 1250
+	1    0    0    -1
+$EndComp
+$Comp
+L power:+3V3 #PWR?
+U 1 1 60F1EB4C
+P 5250 3500
+F 0 "#PWR?" H 5250 3350 50  0001 C CNN
+F 1 "+3V3" V 5265 3628 50  0000 L CNN
+F 2 "" H 5250 3500 50  0001 C CNN
+F 3 "" H 5250 3500 50  0001 C CNN
+	1    5250 3500
+	0    1    1    0
+$EndComp
+$Comp
+L power:+3V3 #PWR?
+U 1 1 60F24168
+P 6100 2900
+F 0 "#PWR?" H 6100 2750 50  0001 C CNN
+F 1 "+3V3" V 6115 3028 50  0000 L CNN
+F 2 "" H 6100 2900 50  0001 C CNN
+F 3 "" H 6100 2900 50  0001 C CNN
+	1    6100 2900
+	0    -1   -1   0
+$EndComp
 $EndSCHEMATC

Commit message: wiring in progress
Parts:
- added C? (x2): 30p, symbol Device:C
- added Y?: Crystal_GND24, symbol Device:Crystal_GND24
Connections:
- net +3V3: now also U?.20 (VCC-IO), U?.5 (VCC-IO)
- net GND: now also J?.9 (SHIELD), C?.2, C?.2, Y?.2, Y?.4
- net CLKN: now reaches U?.51 (HOSCI)
- net CLKN: now also C?.1, Y?.3
- net CLKP: now reaches U?.52 (HOSCO)
- net CLKP: now also C?.1, Y?.1
- no-connect marks 42 -> 41
Other:
- moved on the sheet: J?

Commit message: wiring in progress ..
Parts:
- added C1, C2, C3: 220p, Capacitor_SMD:C_0402_1005Metric_Pad0.74x0.62mm_HandSolder, symbol Device:C
- added C10: 1u, Capacitor_SMD:C_0402_1005Metric_Pad0.74x0.62mm_HandSolder, symbol Device:C
- added C4, C5, C6, C7, C8, C9: 10u, Capacitor_SMD:C_0402_1005Metric_Pad0.74x0.62mm_HandSolder, symbol Device:C
- added J1: Conn_01x02_Male, Connector_PinHeader_1.27mm:PinHeader_1x02_P1.27mm_Vertical, symbol Connector:Conn_01x02_Male
- added L1, L2, L3: 1.5u, Inductor_SMD:L_0402_1005Metric_Pad0.77x0.64mm_HandSolder, symbol Device:L
- added R1, R2, R3, R4, R5, R6: 100k, Resistor_SMD:R_0402_1005Metric_Pad0.72x0.64mm_HandSolder, symbol Device:R
- added R7: R, Resistor_SMD:R_0402_1005Metric_Pad0.72x0.64mm_HandSolder, symbol Device:R
- added R8, R9: 2k2, Resistor_SMD:R_0402_1005Metric_Pad0.72x0.64mm_HandSolder, symbol Device:R
- added U2: EA3036, Package_DFN_QFN:QFN-20-1EP_3x3mm_P0.45mm_EP1.6x1.6mm, symbol PumpkinPi:EA3036
- C11, C12: renamed from C?; footprint (none) -> Capacitor_SMD:C_0402_1005Metric_Pad0.74x0.62mm_HandSolder
- J2: renamed from J?; footprint (none) -> Connector_PinHeader_2.54mm:PinHeader_1x04_P2.54mm_Vertical
- J3: renamed from J?; footprint (none) -> Connector_PinHeader_1.27mm:PinHeader_1x09_P1.27mm_Vertical
- U1: renamed from U?; footprint (none) -> PumpkinPi:QFN-88_EP_10x10_Pitch0.4mm
- Y1: renamed from Y?; footprint (none) -> Crystal:Crystal_SMD_2016-4Pin_2.0x1.6mm
Connections:
- net +1V1: now also C1.1, C4.1, L1.1, R1.1
- net +2V5: now also U1.80 (AVCC), C2.1, C5.1, L2.1, R3.1, R8.1
- net +3V3: now also U1.4 (HPVCC), U1.67 (UVCC), U1.73 (TV_VCC), C3.1, C6.1, L3.1, R5.1, R7.1
- net GND: now also U1.74 (TVGND), U1.82 (AGND), C1.2, C10.2, C2.2, C3.2, C4.2, C5.2, C6.2, C7.2, C8.2, C9.1, J1.1 (Pin_1), R1.2, R2.1, R2.2, R3.2, R4.1, R4.2, R5.2, R6.1, R6.2, R9.2, U2.1 (GND3), U2.12 (GND1), U2.13 (GND1), U2.14 (FB1), U2.15 (AGND), U2.17 (AGND), U2.4 (GND2), U2.5 (GND2)
- net USB_VBUS: now also C10.1, C7.1, C8.1, C9.2, U2.10 (VIN1), U2.16 (VCC), U2.18 (EN3), U2.19 (VIN3), U2.7 (VIN2), U2.8 (EN2), U2.9 (EN1)
- net SVREF: now reaches U1.33 (SVREF)
- net SVREF: now also R8.2, R9.1
- net SDA: now reaches U1.37 (PE12)
- net SCL: now reaches U1.38 (PE11)
- net SPI_CLK: now reaches U1.59 (PC0)
- net SPI_CS: now reaches U1.60 (PC1)
- net SPI_MISO: now reaches U1.61 (PC2)
- net SPI_MOSI: now reaches U1.62 (PC3)
- net RESET: now reaches U1.70 (RESET)
- net RESET: now also J1.2 (Pin_2), R7.2
- new net FB2: U2.3 (FB2)
- new net FB3: U2.2 (FB3)
- new net LX1: L1.2, L2.2, L3.2, U2.11 (LX1)
- new net LX2: U2.6 (LX2)
- new net LX3: U2.20 (LX3)

Commit message: progress on wiring
Connections:
- net GND: no longer C1.2, C2.2, C3.2, R1.2, R2.1, R3.2, R4.1, R5.2, R6.1, U2.14 (FB1)
- new net FB1: C1.2, C2.2, C3.2, R1.2, R2.1, R3.2, R4.1, R5.2, R6.1, U2.14 (FB1)
Changed lines of the file:
@@
 Wire Wire Line
 	1000 6100 1300 6100
-Connection ~ 1700 6100
 Connection ~ 1300 6100
-Wire Wire Line
-	1300 6100 1700 6100
 Wire Wire Line
 	1000 5800 1300 5800
@@
 Wire Wire Line
 	1000 7050 1300 7050
-Connection ~ 1700 7050
 Connection ~ 1300 7050
-Wire Wire Line
-	1300 7050 1700 7050
 Wire Wire Line
 	1000 6750 1300 6750
@@
 Wire Wire Line
 	1000 5200 1300 5200
-Connection ~ 1700 5200
 Connection ~ 1300 5200
 Wire Wire Line
-	1300 5200 1700 5200
-Wire Wire Line
 	1000 4900 1300 4900

Commit message: wiring in progress
Connections:
- net FB1: no longer C2.2, C3.2, R3.2, R4.1, R5.2, R6.1
- net FB2: now also C2.2, R3.2, R4.1
- net FB3: now also C3.2, R5.2, R6.1
- net LX1: no longer L2.2, L3.2
- net LX2: now also L2.2
- net LX3: now also L3.2
Changed lines of the file:
@@
 	1300 5800 1700 5800
 Text Label 700  5800 2    50   ~ 0
-LX1
+LX2
 Text Label 700  6100 2    50   ~ 0
-FB1
+FB2
 Wire Wire Line
 	700  6100 1000 6100
@@
 	1300 6750 1700 6750
 Text Label 700  6750 2    50   ~ 0
-LX1
+LX3
 Text Label 700  7050 2    50   ~ 0
-FB1
+FB3
 Wire Wire Line
 	700  7050 1000 7050

Commit message: progress ...
Parts:
- J1: footprint Connector_PinHeader_1.27mm:PinHeader_1x02_P1.27mm_Vertical -> Connector_PinHeader_1.27mm:PinHeader_1x02_P1.27mm_Vertical_SMD_Pin1Left
Changed lines of the file:
@@
 F 0 "J1" H 5972 1582 50  0000 R CNN
 F 1 "Conn_01x02_Male" H 5972 1673 50  0000 R CNN
-F 2 "Connector_PinHeader_1.27mm:PinHeader_1x02_P1.27mm_Vertical" H 6000 1700 50  0001 C CNN
+F 2 "Connector_PinHeader_1.27mm:PinHeader_1x02_P1.27mm_Vertical_SMD_Pin1Left" H 6000 1700 50  0001 C CNN
 F 3 "~" H 6000 1700 50  0001 C CNN
 	1    6000 1700

Commit message: huge progress
Parts:
- removed C1, C2, C3: 220p, Capacitor_SMD:C_0402_1005Metric_Pad0.74x0.62mm_HandSolder, symbol Device:C
- removed C10: 1u, Capacitor_SMD:C_0402_1005Metric_Pad0.74x0.62mm_HandSolder, symbol Device:C
- removed C4, C5, C6, C7, C8, C9: 10u, Capacitor_SMD:C_0402_1005Metric_Pad0.74x0.62mm_HandSolder, symbol Device:C
- removed L1, L2, L3: 1.5u, Inductor_SMD:L_0402_1005Metric_Pad0.77x0.64mm_HandSolder, symbol Device:L
- removed R1, R2, R3, R4, R5, R6: 100k, Resistor_SMD:R_0402_1005Metric_Pad0.72x0.64mm_HandSolder, symbol Device:R
- removed U2: EA3036, Package_DFN_QFN:QFN-20-1EP_3x3mm_P0.45mm_EP1.6x1.6mm, symbol PumpkinPi:EA3036
- added C? (x3): 1u, Capacitor_SMD:C_0402_1005Metric_Pad0.74x0.62mm_HandSolder, symbol Device:C
- added J?: 0475710001, MOLEX_0475710001, symbol PumpkinPi:0475710001
- added U? (x3): TPS717xx, Package_TO_SOT_SMD:SOT-353_SC-70-5_Handsoldering, symbol PumpkinPi:TPS717xx
- R7: value R -> 51k
- Y1: footprint Crystal:Crystal_SMD_2016-4Pin_2.0x1.6mm -> Crystal:Crystal_SMD_5032-4Pin_5.0x3.2mm
Connections:
- net +1V1: now also C?.1, U?.5 (OUT)
- net +2V5: now also C?.1, U?.5 (OUT)
- net +3V3: now also C?.1, U?.5 (OUT)
- net GND: now also C?.2, C?.2, C?.2, U?.2 (GND), U?.2 (GND), U?.2 (GND)
- net USB_VBUS: now also U?.1 (IN), U?.1 (IN), U?.1 (IN), U?.3 (EN), U?.3 (EN), U?.3 (EN)
- no-connect marks 41 -> 44

Commit message: schemqtic finished, routing started
Parts:
- removed J3: Micro_SD_Card, Connector_PinHeader_1.27mm:PinHeader_1x09_P1.27mm_Vertical, symbol Connector:Micro_SD_Card
- J1: footprint Connector_PinHeader_1.27mm:PinHeader_1x02_P1.27mm_Vertical_SMD_Pin1Left -> Connector_PinHeader_1.00mm:PinHeader_1x02_P1.00mm_Vertical
- U2, U3, U4: renamed from U?; footprint Package_TO_SOT_SMD:SOT-353_SC-70-5_Handsoldering -> Package_TO_SOT_SMD:SOT-353_SC-70-5
- gave numbers to parts that had none: 4
Connections:
- net +2V5: now also C2.1, U3.5 (OUT); no longer C3.1, U4.5 (OUT)
- net +3V3: now also C3.1, J3.4 (VDD), U4.5 (OUT); no longer C2.1, U3.5 (OUT)
- net GND: now also J3.10 (GND@2), J3.13 (GND@3), J3.6 (VSS), J3.9 (GND@1)
- net SD0_CLK: now also J3.5 (CLK)
- net SD0_CMD: now also J3.3 (CMD)
- net SD0_D0: now also J3.7 (DAT0)
- net SD0_D1: now also J3.8 (DAT1)
- net SD0_D2: now also J3.1 (DAT2)
- net SD0_D3: now also J3.2 (DAT3/CD)
- net PD7: now reaches U1.13 (PD7)
- net PD8: now reaches U1.14 (PD8)
- net PD9: now reaches U1.15 (PD9)
- net PD10: now reaches U1.16 (PD10)
- no-connect marks 44 -> 43
Other:
- moved on the sheet: J1, J3, R7, R8, R9
