File: Hardware/PumpkinPi.BAK.kicad_pcb (KiCad board)
At the start: 2 copper layers, 12.1 x 13.3 mm, 30 parts, among them J1 Conn_01x02_Male, J2 Conn_01x04, J3 Micro_SD_Card, U1 F1C100s, U2 EA3036, Y1 Crystal_GND24

Commit message: progress ...
Parts:
- moved C4 20.6 mm to (105.9, 86.5), turned to 90 degrees
- moved R2 20.3 mm to (105.0, 86.5), turned to 270 degrees
- moved R1 17.4 mm to (106.8, 86.5), turned to 90 degrees
- moved U1 16.0 mm to (90.0, 91.2)
- moved L1 14.1 mm to (108.5, 87.0)
- moved C1 14.0 mm to (108.5, 86.0), turned to 180 degrees
- moved J1 12.5 mm to (94.2, 81.9)
- moved R7 9.96 mm to (92.2, 82.7)
- moved C8 5.22 mm to (110.8, 86.6)
- moved C10 5.22 mm to (110.8, 89.2)
- moved C7 5.22 mm to (110.8, 85.3)
- moved C9 5.22 mm to (110.8, 87.9)
- moved U2 1.65 mm to (106.9, 89.7), turned to 90 degrees
Routing:
- net /USB_DM: track 7.31 -> 0.00 mm, vias 1 -> 0
- net /USB_VBUS: track 3.81 -> 9.61 mm
- net /RESET: track 4.55 -> 0.00 mm, vias 1 -> 0
- net +1V1: track 5.83 -> 1.92 mm
- net /USB_DP: track 4.46 -> 0.56 mm, vias 1 -> 0
- net GND: track 9.50 -> 11.9 mm
- net +3V3: track 1.99 -> 0.00 mm, vias 1 -> 0
- net /LX1: track 0.00 -> 1.24 mm
- net /FB1: track 2.37 -> 3.59 mm

Commit message: Updated to KiCAD 6
Other:
- net class Default removed
